File: Hardware/Intar_IR_LED_Module/Intar_IR_LED_Module.brd (EAGLE design)
At the start: 25.8 x 22.4 mm, 19 parts, among them J1 GROVE-4P-2.0-3470130P1, Q1 MMBT2222A, Q2 MMBT2222A

Commit message: Created BOM
Parts:
- C1: value 10nF -> DNP
- R1: value 30? -> 33
Changed lines of the file:
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@@
 <setting verticaltext="up"/>
 </settings>
-<grid distance="1" unitdist="mm" unit="mm" style="dots" multiple="1" display="yes" altdistance="1" altunitdist="inch" altunit="inch"/>
+<grid distance="1" unitdist="mm" unit="mm" style="dots" multiple="1" display="yes" altdistance="0.005" altunitdist="inch" altunit="inch"/>
 <layers>
 <layer number="1" name="Top" color="4" fill="1" visible="yes" active="yes"/>
@@
 <layer number="45" name="Holes" color="7" fill="1" visible="yes" active="yes"/>
 <layer number="46" name="Milling" color="3" fill="1" visible="no" active="yes"/>
-<layer number="47" name="Measures" color="7" fill="1" visible="yes" active="yes"/>
+<layer number="47" name="Measures" color="7" fill="1" visible="no" active="yes"/>
 <layer number="51" name="tDocu" color="6" fill="1" visible="yes" active="yes"/>
 <layer number="52" name="bDocu" color="7" fill="1" visible="no" active="yes"/>
@@
 </autorouter>
 <elements>
-<element name="C1" library="SparkFun-Capacitors" package="0603-CAP" value="10nF" x="6.35" y="1.905" rot="R270">
+<element name="C1" library="SparkFun-Capacitors" package="0603-CAP" value="DNP" x="6.35" y="1.905" rot="R270">
 <attribute name="PROD_ID" value="CAP-00867" x="6.35" y="1.905" size="1.778" layer="27" rot="R270" display="off"/>
 </element>
@@
 <attribute name="PROD_ID" value="TRANS-08049" x="3.175" y="5.08" size="1.778" layer="27" rot="R90" display="off"/>
 </element>
-<element name="R1" library="SparkFun-Resistors" package="0603-RES" value="30?" x="-6.35" y="-1.905" rot="R90"/>
+<element name="R1" library="SparkFun-Resistors" package="0603-RES" value="33" x="-6.35" y="-1.905" rot="R90"/>
 <element name="R2" library="SparkFun-Resistors" package="0603-RES" value="2.2k" x="-6.35" y="1.905" rot="R90">
 <attribute name="PROD_ID" value="RES-08272" x="-6.35" y="1.905" size="1.778" layer="27" rot="R90" display="off"/>
