File: Hardware/Intar_IR_Module/Intar_IR_Module.sch (EAGLE design)
At the start: 19 parts, among them J2 GROVE-4P-2.0-3470130P1, Q1 MMBT2222A, Q2 MMBT2222A

Commit message: Imported logo into Eagle
Parts:
- added U$1: LOGOSM, Intar_Eagle_Library:LOGOSM
Changed lines of the file:
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@@
 <setting verticaltext="up"/>
 </settings>
-<grid distance="0.1" unitdist="inch" unit="inch" style="lines" multiple="1" display="yes" altdistance="0.01" altunitdist="inch" altunit="inch"/>
+<grid distance="0.1" unitdist="inch" unit="inch" style="lines" multiple="1" display="no" altdistance="0.01" altunitdist="inch" altunit="inch"/>
 <layers>
 <layer number="1" name="Top" color="4" fill="1" visible="no" active="no"/>
@@
 <part name="GND5" library="SparkFun-Aesthetics" deviceset="GND" device=""/>
 <part name="SUPPLY5" library="SparkFun-Aesthetics" deviceset="VCC" device=""/>
+<part name="U$1" library="Intar_Eagle_Library" deviceset="LOGO" device="SM"/>
 </parts>
 <sheets>
@@
 <instance part="GND5" gate="1" x="81.28" y="149.86"/>
 <instance part="SUPPLY5" gate="G$1" x="88.9" y="147.32"/>
+<instance part="U$1" gate="G$1" x="104.14" y="2.54"/>
 </instances>
 <busses>

Commit message: Finished RGB and IR modules
Parts:
- renumbered J2 to J1
Connections:
- net GND: now also J1.4; no longer J1.1
- net IR: now also J1.2; no longer J1.3
- net LEDS: now also J1.1; no longer J1.4
- net VCC: now also J1.3; no longer J1.2
Other:
- note added: "v02"
- note removed: "v01"
Changed lines of the file:
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@@
 <setting verticaltext="up"/>
 </settings>
-<grid distance="0.1" unitdist="inch" unit="inch" style="lines" multiple="1" display="no" altdistance="0.01" altunitdist="inch" altunit="inch"/>
+<grid distance="0.1" unitdist="inch" unit="inch" style="lines" multiple="1" display="yes" altdistance="0.01" altunitdist="inch" altunit="inch"/>
 <layers>
 <layer number="1" name="Top" color="4" fill="1" visible="no" active="no"/>
@@
 <part name="STANDOFF2" library="SparkFun-Electromechanical" deviceset="STAND-OFF" device=""/>
 <part name="LOGO1" library="SparkFun-Aesthetics" deviceset="OSHW-LOGO" device="S"/>
-<part name="J2" library="Connector" deviceset="GROVE-4P-2.0" device="-3470130P1"/>
 <part name="GND5" library="SparkFun-Aesthetics" deviceset="GND" device=""/>
 <part name="SUPPLY5" library="SparkFun-Aesthetics" deviceset="VCC" device=""/>
 <part name="U$1" library="Intar_Eagle_Library" deviceset="LOGO" device="SM"/>
+<part name="J1" library="Connector" deviceset="GROVE-4P-2.0" device="-3470130P1"/>
 </parts>
 <sheets>
@@
 <plain>
 <text x="155.956" y="6.35" size="2.54" layer="94">Shawn Hymel</text>
-<text x="238.76" y="7.62" size="2.54" layer="94">v01</text>
+<text x="238.76" y="7.62" size="2.54" layer="94">v02</text>
 <text x="66.04" y="135.89" size="1.778" layer="97">Grove</text>
 <text x="190.5" y="93.98" size="1.778" layer="97">Cut jumper to
@@
 <instance part="STANDOFF2" gate="G$1" x="241.3" y="27.94"/>
 <instance part="LOGO1" gate="G$1" x="132.08" y="10.16"/>
-<instance part="J2" gate="J" x="68.58" y="143.51" smashed="yes">
-<attribute name="NAME" x="66.04" y="149.352" size="1.27" layer="95" ratio="10"/>
-</instance>
 <instance part="GND5" gate="1" x="81.28" y="149.86"/>
 <instance part="SUPPLY5" gate="G$1" x="88.9" y="147.32"/>
 <instance part="U$1" gate="G$1" x="104.14" y="2.54"/>
+<instance part="J1" gate="J" x="68.58" y="143.51" smashed="yes" rot="MR180">
+<attribute name="NAME" x="66.04" y="149.352" size="1.27" layer="95" ratio="10"/>
+</instance>
 </instances>
 <busses>
@@
 </segment>
 <segment>
-<pinref part="J2" gate="J" pin="1"/>
 <wire x1="73.66" y1="147.32" x2="76.2" y2="147.32" width="0.1524" layer="91"/>
 <wire x1="76.2" y1="147.32" x2="76.2" y2="154.94" width="0.1524" layer="91"/>
@@
 <wire x1="81.28" y1="154.94" x2="81.28" y2="152.4" width="0.1524" layer="91"/>
 <pinref part="GND5" gate="1" pin="GND"/>
+<pinref part="J1" gate="J" pin="4"/>
 </segment>
 </net>
@@
 </segment>
 <segment>
-<pinref part="J2" gate="J" pin="2"/>
 <wire x1="73.66" y1="144.78" x2="88.9" y2="144.78" width="0.1524" layer="91"/>
 <wire x1="88.9" y1="144.78" x2="88.9" y2="147.32" width="0.1524" layer="91"/>
 <pinref part="SUPPLY5" gate="G$1" pin="VCC"/>
+<pinref part="J1" gate="J" pin="3"/>
 </segment>
 </net>
@@
 </segment>
 <segment>
-<pinref part="J2" gate="J" pin="3"/>
 <wire x1="73.66" y1="142.24" x2="76.2" y2="142.24" width="0.1524" layer="91"/>
 <label x="76.2" y="142.24" size="1.27" layer="95" xref="yes"/>
+<pinref part="J1" gate="J" pin="2"/>
 </segment>
 </net>
@@
 </segment>
 <segment>
-<pinref part="J2" gate="J" pin="4"/>
 <wire x1="73.66" y1="139.7" x2="76.2" y2="139.7" width="0.1524" layer="91"/>
 <label x="76.2" y="139.7" size="1.27" layer="95" xref="yes"/>
+<pinref part="J1" gate="J" pin="1"/>
 </segment>
 </net>
